Commit message: Add base link, right and left wheel

File: my_rb1_description/urdf/my_rb1_robot.urdf (robot description, URDF)
Before this commit: robot rb1_robot, 7 links, 6 joints
Links:
- removed link back_caster
- removed link front_caster
- removed link front_laser
- link base_link: mass None -> 18; geometry collision cylinder length=0.3 radius=0.25; visual cylinder length=0.3 radius=0.25
- link left_wheel: mass None -> 1.5; geometry collision cylinder length=0.05 radius=0.025; visual cylinder length=0.05 radius=0.025
- link right_wheel: mass None -> 1.5; geometry collision cylinder length=0.05 radius=0.025; visual cylinder length=0.05 radius=0.025
Joints:
- removed joint base_link_back_caster_joint
- removed joint base_link_front_caster_joint
- removed joint base_link_front_laser_joint
- joint base_link_left_wheel_joint: axis (none) -> 0 1 0; child (none) -> left_wheel; origin (none) -> xyz=0 0.2 -0.15 rpy=0 0 0; parent (none) -> base_link; type  -> continuous
- joint base_link_plate_joint: child (none) -> base_link; origin (none) -> xyz=0 0 0 rpy=0 0 0; parent (none) -> base_footprint; type  -> fixed
- joint base_link_right_wheel_joint: axis (none) -> 0 1 0; child (none) -> right_wheel; origin (none) -> xyz=0 -0.2 -0.15 rpy=0 0 0; parent (none) -> base_link; type  -> continuous

Commit message: Add casters and laser link

File: my_rb1_description/urdf/my_rb1_robot.urdf (robot description, URDF)
Before this commit: robot rb1_robot, 4 links, 3 joints
Links:
- added link back_caster, mass 1; collision cylinder length=0.03 radius=0.025; visual cylinder length=0.03 radius=0.025
- added link front_caster, mass 1; collision cylinder length=0.03 radius=0.025; visual cylinder length=0.03 radius=0.025
- added link front_laser, mass 3
Joints:
- added joint base_link_back_caster_joint: type fixed, parent base_link, child back_caster, origin xyz=-0.1 0 -0.15 rpy=0 0 0
- added joint base_link_front_caster_joint: type fixed, parent base_link, child front_caster, origin xyz=0.1 0 -0.15 rpy=0 0 0
- added joint base_link_front_laser_joint: type fixed, parent base_link, child front_laser, origin xyz=0.25 0 0.075 rpy=1.5707 0 0

Commit message: Fix laser scan rotation

File: my_rb1_description/urdf/my_rb1_robot.urdf (robot description, URDF)
Before this commit: robot rb1_robot, 7 links, 6 joints
Joints:
- joint base_link_front_laser_joint: origin xyz=0.25 0 0.075 rpy=1.5707 0 0 -> xyz=0.25 0 0.075 rpy=3.14159 0 0

Commit message: Fix caster link geometry from cylinder to sphere

File: my_rb1_description/urdf/my_rb1_robot.urdf (robot description, URDF)
Before this commit: robot rb1_robot, 7 links, 6 joints
Links:
- link back_caster: mass 1 -> 0.5; geometry collision sphere radius=0.025; visual sphere radius=0.025
- link front_caster: mass 1 -> 0.5; geometry collision sphere radius=0.025; visual sphere radius=0.025

Commit message: Fix base_footprint position

File: my_rb1_description/urdf/my_rb1_robot.urdf (robot description, URDF)
Before this commit: robot rb1_robot, 7 links, 6 joints
Joints:
- joint base_link_plate_joint: origin xyz=0 0 0 rpy=0 0 0 -> xyz=0 0 0.15 rpy=0 0 0
